File: PCB/_saved_Compuboard.sch (KiCad schematic (older format))
At the start: 64 parts, among them SW0 SW_PUSH, SW0:0 SWITCH_DIODE, SW0:1 SWITCH_DIODE, SW0:10 SWITCH_DIODE, SW0:11 SWITCH_DIODE, SW0:12 SWITCH_DIODE, SW0:13 SWITCH_DIODE, SW0:2 SWITCH_DIODE, SW0:3 SWITCH_DIODE, SW0:4 SWITCH_DIODE, SW0:5 SWITCH_DIODE, SW0:6 SWITCH_DIODE, SW0:7 SWITCH_DIODE, SW0:8 SWITCH_DIODE, SW0:9 SWITCH_DIODE, SW1:0 SWITCH_DIODE, SW1:1 SWITCH_DIODE, SW1:10 SWITCH_DIODE, SW1:11 SWITCH_DIODE, SW1:12 SWITCH_DIODE, SW1:13 SWITCH_DIODE, SW1:2 SWITCH_DIODE, SW1:3 SWITCH_DIODE, SW1:4 SWITCH_DIODE, SW1:5 SWITCH_DIODE, SW1:6 SWITCH_DIODE, SW1:7 SWITCH_DIODE, SW1:8 SWITCH_DIODE, SW1:9 SWITCH_DIODE, SW2:0 SWITCH_DIODE, SW2:1 SWITCH_DIODE, SW2:10 SWITCH_DIODE, SW2:11 SWITCH_DIODE, SW2:13 SWITCH_DIODE, SW2:2 SWITCH_DIODE, SW2:3 SWITCH_DIODE, SW2:4 SWITCH_DIODE, SW2:5 SWITCH_DIODE, SW2:6 SWITCH_DIODE, SW2:7 SWITCH_DIODE, SW2:8 SWITCH_DIODE, SW2:9 SWITCH_DIODE, SW3:0 SWITCH_DIODE, SW3:10 SWITCH_DIODE, SW3:11 SWITCH_DIODE, SW3:13 SWITCH_DIODE, SW3:2 SWITCH_DIODE, SW3:3 SWITCH_DIODE, SW3:4 SWITCH_DIODE, SW3:5 SWITCH_DIODE, SW3:6 SWITCH_DIODE, SW3:7 SWITCH_DIODE, SW3:8 SWITCH_DIODE, SW3:9 SWITCH_DIODE, SW4:0 SWITCH_DIODE, SW4:1 SWITCH_DIODE, SW4:10 SWITCH_DIODE, SW4:11 SWITCH_DIODE, SW4:12 SWITCH_DIODE, SW4:13 SWITCH_DIODE, SW4:3 SWITCH_DIODE, SW4:6 SWITCH_DIODE

Commit message: Add better TTY font
Parts:
- gave numbers to parts that had none: 1
Changed lines of the file:
@@
 ROW4
 $Comp
-L 74LS151 U?
+L 74LS151 U0
 U 1 1 5C30F3BE
 P 8050 5500
-F 0 "U?" H 8050 5500 50  0000 C CNN
+F 0 "U0" H 8050 5500 50  0000 C CNN
 F 1 "74LS151" H 8050 5350 50  0000 C CNN
 F 2 "" H 8050 5500 50  0001 C CNN
@@
 SEL
 $Comp
-L GND #PWR?
+L GND #PWR06
 U 1 1 5C334ABC
 P 8750 5100
-F 0 "#PWR?" H 8750 4850 50  0001 C CNN
+F 0 "#PWR06" H 8750 4850 50  0001 C CNN
 F 1 "GND" H 8750 4950 50  0000 C CNN
 F 2 "" H 8750 5100 50  0001 C CNN
@@
 $EndComp
 $Comp
-L VCC #PWR?
+L VCC #PWR07
 U 1 1 5C334C90
 P 8750 5000
-F 0 "#PWR?" H 8750 4850 50  0001 C CNN
+F 0 "#PWR07" H 8750 4850 50  0001 C CNN
 F 1 "VCC" H 8750 5150 50  0000 C CNN
 F 2 "" H 8750 5000 50  0001 C CNN
