File: PCB/Compuboard.kicad_pcb (KiCad board)
At the start: 2 copper layers, 290.8 x 125.1 mm, 64 parts, among them SW0 SW_PUSH, SW0:0 SWITCH_DIODE, SW0:1 SWITCH_DIODE, SW0:10 SWITCH_DIODE, SW0:11 SWITCH_DIODE, SW0:12 SWITCH_DIODE, SW0:13 SWITCH_DIODE, SW0:2 SWITCH_DIODE, SW0:3 SWITCH_DIODE, SW0:4 SWITCH_DIODE, SW0:5 SWITCH_DIODE, SW0:6 SWITCH_DIODE, SW0:7 SWITCH_DIODE, SW0:8 SWITCH_DIODE, SW0:9 SWITCH_DIODE, SW1:0 SWITCH_DIODE, SW1:1 SWITCH_DIODE, SW1:10 SWITCH_DIODE, SW1:11 SWITCH_DIODE, SW1:12 SWITCH_DIODE, SW1:13 SWITCH_DIODE, SW1:2 SWITCH_DIODE, SW1:3 SWITCH_DIODE, SW1:4 SWITCH_DIODE, SW1:5 SWITCH_DIODE, SW1:6 SWITCH_DIODE, SW1:7 SWITCH_DIODE, SW1:8 SWITCH_DIODE, SW1:9 SWITCH_DIODE, SW2:0 SWITCH_DIODE, SW2:1 SWITCH_DIODE, SW2:10 SWITCH_DIODE, SW2:11 SWITCH_DIODE, SW2:13 SWITCH_DIODE, SW2:2 SWITCH_DIODE, SW2:3 SWITCH_DIODE, SW2:4 SWITCH_DIODE, SW2:5 SWITCH_DIODE, SW2:6 SWITCH_DIODE, SW2:7 SWITCH_DIODE, SW2:8 SWITCH_DIODE, SW2:9 SWITCH_DIODE, SW3:0 SWITCH_DIODE, SW3:10 SWITCH_DIODE, SW3:11 SWITCH_DIODE, SW3:13 SWITCH_DIODE, SW3:2 SWITCH_DIODE, SW3:3 SWITCH_DIODE, SW3:4 SWITCH_DIODE, SW3:5 SWITCH_DIODE, SW3:6 SWITCH_DIODE, SW3:7 SWITCH_DIODE, SW3:8 SWITCH_DIODE, SW3:9 SWITCH_DIODE, SW4:0 SWITCH_DIODE, SW4:1 SWITCH_DIODE, SW4:10 SWITCH_DIODE, SW4:11 SWITCH_DIODE, SW4:12 SWITCH_DIODE, SW4:13 SWITCH_DIODE, SW4:3 SWITCH_DIODE, SW4:6 SWITCH_DIODE, U0 74LS151

Commit message: Add stuff
Parts:
- moved SW0 62.7 mm to (280.9, -143.0)
- moved U0 19.9 mm to (288.0, -114.6), turned to 180 degrees
- moved PM0 16.8 mm to (266.7, -120.7), turned to 270 degrees
Connections:
- PM0 pad 0: /MUL2 -> /COL0
- PM0 pad 1: /MUL1 -> /COL1
- PM0 pad 17: (no net) -> /MUL2
- PM0 pad 18: /COL1 -> /MUL1
- PM0 pad 19: /COL2 -> /MUL0
- PM0 pad 4: /MUL0 -> /COL2
- SW0:0 pad 1: Net-(SW0:0-Pad1) -> /COL0
- SW1:0 pad 1: Net-(SW0:0-Pad1) -> /COL0
- SW2:0 pad 1: Net-(SW0:0-Pad1) -> /COL0
- SW3:0 pad 1: Net-(SW0:0-Pad1) -> /COL0
- SW4:0 pad 1: Net-(SW0:0-Pad1) -> /COL0
Routing:
- net /COL0: track 0.00 -> 391.5 mm, vias 0 -> 2
- net /COL1: track 90.7 -> 382.4 mm, vias 0 -> 2
- net /COL2: track 77.6 -> 329.4 mm, vias 0 -> 2
- net /COL3: track 99.1 -> 321.2 mm, vias 0 -> 2
- net /COL4: track 73.4 -> 270.1 mm, vias 0 -> 2
- net /COL5: track 72.6 -> 244.5 mm, vias 0 -> 2
- net /COL6: track 94.6 -> 238.4 mm, vias 0 -> 2
- net /COL7: track 71.1 -> 212.0 mm, vias 0 -> 2
- net /COL8: track 73.4 -> 188.4 mm, vias 0 -> 2
- net Net-(SW0:0-Pad1): track 100.0 -> 0.00 mm
- net /COL9: track 73.3 -> 165.3 mm, vias 0 -> 2
- net /COL10: track 93.4 -> 163.8 mm, vias 0 -> 2
- net /COL11: track 92.5 -> 141.1 mm, vias 0 -> 2
- net VCC: track 0.00 -> 43.4 mm
- net /COL12: track 87.0 -> 118.7 mm
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- added copper zone on B.Cu, net GND
- added copper zone on F.Cu, net GND
Other:
- board size 290.8 x 125.1 mm -> 290.8 x 139.1 mm
