File: PCB/Compuboard.sch (KiCad schematic (older format))
At the start: 64 parts, among them SW0 SW_PUSH, SW0:0 SWITCH_DIODE, SW0:1 SWITCH_DIODE, SW0:10 SWITCH_DIODE, SW0:11 SWITCH_DIODE, SW0:12 SWITCH_DIODE, SW0:13 SWITCH_DIODE, SW0:2 SWITCH_DIODE, SW0:3 SWITCH_DIODE, SW0:4 SWITCH_DIODE, SW0:5 SWITCH_DIODE, SW0:6 SWITCH_DIODE, SW0:7 SWITCH_DIODE, SW0:8 SWITCH_DIODE, SW0:9 SWITCH_DIODE, SW1:0 SWITCH_DIODE, SW1:1 SWITCH_DIODE, SW1:10 SWITCH_DIODE, SW1:11 SWITCH_DIODE, SW1:12 SWITCH_DIODE, SW1:13 SWITCH_DIODE, SW1:2 SWITCH_DIODE, SW1:3 SWITCH_DIODE, SW1:4 SWITCH_DIODE, SW1:5 SWITCH_DIODE, SW1:6 SWITCH_DIODE, SW1:7 SWITCH_DIODE, SW1:8 SWITCH_DIODE, SW1:9 SWITCH_DIODE, SW2:0 SWITCH_DIODE, SW2:1 SWITCH_DIODE, SW2:10 SWITCH_DIODE, SW2:11 SWITCH_DIODE, SW2:13 SWITCH_DIODE, SW2:2 SWITCH_DIODE, SW2:3 SWITCH_DIODE, SW2:4 SWITCH_DIODE, SW2:5 SWITCH_DIODE, SW2:6 SWITCH_DIODE, SW2:7 SWITCH_DIODE, SW2:8 SWITCH_DIODE, SW2:9 SWITCH_DIODE, SW3:0 SWITCH_DIODE, SW3:10 SWITCH_DIODE, SW3:11 SWITCH_DIODE, SW3:13 SWITCH_DIODE, SW3:2 SWITCH_DIODE, SW3:3 SWITCH_DIODE, SW3:4 SWITCH_DIODE, SW3:5 SWITCH_DIODE, SW3:6 SWITCH_DIODE, SW3:7 SWITCH_DIODE, SW3:8 SWITCH_DIODE, SW3:9 SWITCH_DIODE, SW4:0 SWITCH_DIODE, SW4:1 SWITCH_DIODE, SW4:10 SWITCH_DIODE, SW4:11 SWITCH_DIODE, SW4:12 SWITCH_DIODE, SW4:13 SWITCH_DIODE, SW4:3 SWITCH_DIODE, SW4:6 SWITCH_DIODE

Commit message: Add first traces to PCB
Parts:
- SW0: footprint Keyboards:SW_TH_Tactile_Omron_B3F-10xx -> Buttons_Switches_ThroughHole:SW_TH_Tactile_Omron_B3F-10xx
- SW0:0, SW0:1, SW0:10, SW0:11, SW0:12, SW0:13, SW0:2, SW0:3, SW0:4, SW0:5, SW0:6, SW0:7, SW0:8, SW0:9, SW1:0, SW1:1, SW1:10, SW1:11, SW1:12, SW1:13, SW1:2, SW1:3, SW1:4, SW1:5, SW1:6, SW1:7, SW1:8, SW1:9, SW2:0, SW2:1, SW2:10, SW2:11, SW2:13, SW2:2, SW2:3, SW2:4, SW2:5, SW2:6, SW2:7, SW2:8, SW2:9, SW3:0, SW3:10, SW3:11, SW3:13, SW3:2, SW3:3, SW3:4, SW3:5, SW3:6, SW3:7, SW3:8, SW3:9, SW4:0, SW4:1, SW4:10, SW4:11, SW4:12, SW4:13, SW4:3, SW4:6: footprint Keyboards:SMK_SWITCH_DIODE_1U -> Keyboards:MX_DIODE
- U0: renamed from U?; footprint (none) -> Housings_DIP:DIP-16_W7.62mm
Connections:
- net ROW3: now also SW3:4.4 (K), SW3:5.4 (K), SW3:7.4 (K), SW3:8.4 (K), SW3:9.4 (K)

Commit message: Add stuff
Connections:
- net COL0: now also PM0.0 (PD3), SW0:0.1, SW1:0.1, SW2:0.1, SW3:0.1, SW4:0.1; no longer PM0.17 (PF5)
- net COL1: now also PM0.1 (PD2); no longer PM0.18 (PF6)
- net COL2: now also PM0.4 (PD1); no longer PM0.19 (PF7)
- net MUL0: now also PM0.19 (PF7); no longer PM0.4 (PD1)
- net MUL1: now also PM0.18 (PF6); no longer PM0.1 (PD2)
- net MUL2: now also PM0.17 (PF5); no longer PM0.0 (PD3)
Changed lines of the file:
@@
 Text Label 11050 3600 0    60   ~ 0
 ROW3
-Text Label 3200 7350 0    60   ~ 0
+Text Label 3200 6750 0    60   ~ 0
 COL0
-Text Label 3200 7450 0    60   ~ 0
+Text Label 3200 6650 0    60   ~ 0
 COL1
-Text Label 3200 7550 0    60   ~ 0
+Text Label 3200 6550 0    60   ~ 0
 COL2
 Text Label 3200 5650 0    60   ~ 0
@@
 Text Label 7350 5950 2    60   ~ 0
 MUL2
-Text Label 3200 6550 0    60   ~ 0
+Text Label 3200 7550 0    60   ~ 0
 MUL0
-Text Label 3200 6650 0    60   ~ 0
+Text Label 3200 7450 0    60   ~ 0
 MUL1
-Text Label 3200 6750 0    60   ~ 0
+Text Label 3200 7350 0    60   ~ 0
 MUL2
 Text Label 7350 4850 2    60   ~ 0
@@
 Connection ~ 7150 3600
 Connection ~ 7900 3600
+Text Label 600  850  0    60   ~ 0
+COL0
 $EndSCHEMATC
